File: PCB/main_keyboard/main_keyboard.kicad_pcb (KiCad board)
At the start: 2 copper layers, 309.6 x 95.2 mm, 213 parts, among them J1 Conn_01x05_Pin, U1 ATmega32U4-A

Commit message: leds placed
smd led footprints placed
Parts:
- removed D66, D67, D68: Diode, ScottoKeebs_Components:Diode_SOD-123
- removed REF**: Hotswap_MX_Plated_2.25u, ScottoKeebs_Hotswap:Hotswap_MX_Plated_2.25u
- removed REF**: Hotswap_MX_Plated_2.75u, ScottoKeebs_Hotswap:Hotswap_MX_Plated_2.75u
- removed REF**: Hotswap_MX_Plated_1.00u, ScottoKeebs_Hotswap:Hotswap_MX_Plated_1.00u
- removed REF**: Hotswap_MX_Plated_1.25u, ScottoKeebs_Hotswap:Hotswap_MX_Plated_1.25u
- added C1: 0.1u, Capacitor_SMD:C_01005_0402Metric_Pad0.57x0.30mm_HandSolder, F.Cu at (-103.5, 86.2)
- added C2: 0.1u, Capacitor_SMD:C_01005_0402Metric_Pad0.57x0.30mm_HandSolder, F.Cu at (-103.5, 87.9)
- added C3: 0.1u, Capacitor_SMD:C_01005_0402Metric_Pad0.57x0.30mm_HandSolder, F.Cu at (-103.5, 89.5)
- added C4: 0.1u, Capacitor_SMD:C_01005_0402Metric_Pad0.57x0.30mm_HandSolder, F.Cu at (-103.5, 91.2)
- added C5: 4.7u, Capacitor_SMD:C_0201_0603Metric_Pad0.64x0.40mm_HandSolder, F.Cu at (-103.5, 96.0)
- added C7: 22p, Capacitor_SMD:C_01005_0402Metric_Pad0.57x0.30mm_HandSolder, F.Cu at (-103.5, 92.8)
- added C8: 22p, Capacitor_SMD:C_01005_0402Metric_Pad0.57x0.30mm_HandSolder, F.Cu at (-103.5, 94.5)
- S64: footprint ScottoKeebs_Hotswap:Hotswap_MX_Plated_1.00u -> ScottoKeebs_Hotswap:Hotswap_MX_Plated_1.50u
- moved D69 394.9 mm to (339.7, 54.0)
- moved D99 374.0 mm to (339.7, 73.0)
- moved D126 367.0 mm to (339.7, 130.2), turned to 180 degrees
- moved D71 357.1 mm to (306.4, 54.0), turned to 180 degrees
- moved D127 347.5 mm to (320.7, 130.2), turned to 180 degrees
- moved D98 345.9 mm to (311.1, 73.0)
- moved D125 341.6 mm to (320.7, 111.1)
- moved D100 339.9 mm to (304.0, 92.1), turned to 180 degrees
- moved D72 328.2 mm to (277.8, 54.0), turned to 180 degrees
- moved D128 327.9 mm to (301.6, 130.2), turned to 180 degrees
- moved D97 322.7 mm to (287.3, 73.0)
- moved D73 308.8 mm to (258.8, 54.0), turned to 180 degrees
- moved D101 308.6 mm to (273.1, 92.1), turned to 180 degrees
- moved D124 307.0 mm to (285.0, 111.1)
- moved D96 304.4 mm to (268.3, 73.0)
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Connections:
- D103 pad 4: Net-(D103-DIN) -> Net-(D102-DOUT)
- D104 pad 4: Net-(D102-DOUT) -> Net-(D103-DOUT)
- D105 pad 4: Net-(D103-DOUT) -> Net-(D104-DOUT)
- D106 pad 4: Net-(D104-DOUT) -> Net-(D105-DOUT)
- D107 pad 4: Net-(D105-DOUT) -> Net-(D106-DOUT)
- D108 pad 4: Net-(D106-DOUT) -> Net-(D107-DOUT)
- D109 pad 4: Net-(D107-DOUT) -> Net-(D108-DOUT)
- D110 pad 4: Net-(D108-DOUT) -> Net-(D109-DOUT)
- D111 pad 4: Net-(D109-DOUT) -> Net-(D110-DOUT)
- D112 pad 4: Net-(D110-DOUT) -> Net-(D111-DOUT)
- D113 pad 4: Net-(D111-DOUT) -> Net-(D112-DOUT)
- D114 pad 4: Net-(D112-DOUT) -> Net-(D113-DOUT)
- D115 pad 4: Net-(D113-DOUT) -> Net-(D114-DOUT)
- D116 pad 4: Net-(D114-DOUT) -> Net-(D115-DOUT)
- D117 pad 4: Net-(D115-DOUT) -> Net-(D116-DOUT)
- D118 pad 4: Net-(D116-DOUT) -> Net-(D117-DOUT)
- D119 pad 4: Net-(D117-DOUT) -> Net-(D118-DOUT)
- D120 pad 4: Net-(D118-DOUT) -> Net-(D119-DOUT)
- D121 pad 4: Net-(D119-DOUT) -> Net-(D120-DOUT)
- D122 pad 4: Net-(D120-DOUT) -> Net-(D121-DOUT)
- D123 pad 4: Net-(D121-DOUT) -> Net-(D122-DOUT)
- D124 pad 4: Net-(D122-DOUT) -> Net-(D123-DOUT)
- D125 pad 4: Net-(D123-DOUT) -> Net-(D124-DOUT)
- D126 pad 4: Net-(D124-DOUT) -> Net-(D125-DOUT)
- D127 pad 4: Net-(D125-DOUT) -> Net-(D126-DOUT)
- D128 pad 4: Net-(D126-DOUT) -> Net-(D127-DOUT)
- D129 pad 4: Net-(D127-DOUT) -> Net-(D128-DOUT)
- D130 pad 4: Net-(D128-DOUT) -> Net-(D129-DOUT)
- D131 pad 4: Net-(D129-DOUT) -> Net-(D130-DOUT)
- D132 pad 2: Net-(D103-DIN) -> Net-(D132-DOUT)
- D132 pad 4: Net-(D130-DOUT) -> Net-(D131-DOUT)
- D133 pad 4: Net-(D131-DOUT) -> Net-(D132-DOUT)
- U1 pad 16: unconnected-(U1-XTAL2-Pad16) -> Net-(U1-XTAL2)
- U1 pad 17: unconnected-(U1-XTAL1-Pad17) -> Net-(U1-XTAL1)
